File: UINIO-Monitor.kicad_pcb (KiCad board)
At the start: 2 copper layers, 66.3 x 77.9 mm, 44 parts, among them J1 Conn_01x09_Male, J2 Conn_01x09_Male, J3 Conn_01x04_Male, P1 LCD_Pad_10Pin, P2 LCD_Pad_12Pin, P3 OLED_Pad_30Pin, U1 ME6211, U2 ME6211, U3 XC6206PxxxMR

Commit message: Release UINIO-Monitor version 2.0.0.
Parts:
- moved ? 0.13 mm to (163.9, 133.9)
Routing:
- net GND: track 96.8 -> 101.5 mm, vias 20 -> 23
- net /3.3V_1.3inch: track 46.8 -> 45.9 mm
- net /SDA_0.96inch: track 17.3 -> 16.4 mm
- net /CS_1.3inch: track 27.2 -> 26.6 mm
Other:
- outline, holes or cut-outs redrawn
- board text added: "Version 2.0.0"
- board text removed: "Version 1.0.0"

Commit message: Update PCB.
Parts:
- moved C4 0.37 mm to (127.7, 117.4)
- moved U2 0.37 mm to (124.2, 117.3)
- moved C6 0.37 mm to (120.7, 117.4)
- moved P2 0.31 mm to (134.4, 128.9), turned to 180 degrees
- moved ? 0.20 mm to (164.0, 123.3)
- moved FPC1 0.10 mm to (122.9, 126.0)
Routing:
- net GND: track 101.5 -> 119.2 mm, vias 23 -> 21
- net /5V_1.3inch: track 33.7 -> 43.0 mm, vias 2 -> 1
- net /3.3V_1.3inch: track 45.9 -> 54.9 mm
- net Net-(P2-Pad2): track 13.5 -> 6.30 mm, vias 2 -> 0
- net /RESET_1.3inch: track 28.8 -> 23.2 mm, vias 2 -> 0
- net /BLK_1.3inch: track 23.5 -> 28.7 mm
- net /SCL_1.3inch: track 23.7 -> 22.3 mm
- net /SDA_1.3inch: track 24.1 -> 22.7 mm, vias 0 -> 2
- net /CS_1.3inch: track 26.6 -> 26.5 mm, vias 0 -> 2

Commit message: Update board frame.
Parts:
- added ?: LOGO, LOGO, F.Cu at (96.3, 93.2)
Other:
- board size 66.3 x 77.9 mm -> 90.8 x 77.9 mm

Commit message: Update PCB.
Parts:
- added ?: LOGO, LOGO, B.Cu at (96.3, 93.2)
- added C14: 1uF, Capacitor_SMD:C_0402_1005Metric, F.Cu at (58.2, 71.8)
- added C15: 1uF, Capacitor_SMD:C_0402_1005Metric, F.Cu at (58.2, 69.8)
- added C16: 1uF, Capacitor_SMD:C_0402_1005Metric, F.Cu at (60.8, 88.2)
- added J4: Conn_01x09_Male, Connector_PinHeader_2.54mm:PinHeader_1x09_P2.54mm_Vertical, F.Cu at (87.9, 68.0)
- added P4: LCD_Pad_13Pin, Uinio:LCD_Pad_13Pin, F.Cu at (97.2, 78.9)
- added R11: 10K, Resistor_SMD:R_0402_1005Metric, F.Cu at (63.1, 80.5)
- added R12: 1K, Resistor_SMD:R_0402_1005Metric, F.Cu at (74.4, 80.6)
- added R13: 10R, Resistor_SMD:R_0402_1005Metric, F.Cu at (65.7, 88.4)
- added U4: ME6211, Uinio:SOT-23-5_L3.0-W1.7-P0.95-LS2.8-BR, F.Cu at (61.9, 70.4)
- added VT3: S8050, Uinio:SOT-23-3_L2.9-W1.6-P1.90-LS2.9-BL, F.Cu at (74.0, 73.5)
Connections:
- net /RESET_0.96inch renamed /RESET_0.96_OLED
- net /SCK_0.96inch renamed /SCK_0.96_OLED
- net /SDA_0.96inch renamed /SDA_0.96_OLED
- net /VCC_0.96inch renamed /VCC_0.96_OLED
- C8 pad 2: /3.3V_0.96inch -> /3.3V_OLED
- C9 pad 2: /3.3V_0.96inch -> /3.3V_OLED
- D1 pad 1: /3.3V_0.96inch -> /3.3V_OLED
- FPC3 pad 4: /3.3V_0.96inch -> /3.3V_0.96_OLED
- P3 pad 11: /3.3V_0.96inch -> /3.3V_OLED
- P3 pad 6: /3.3V_0.96inch -> /3.3V_OLED
- P3 pad 9: /3.3V_0.96inch -> /3.3V_OLED
- R7 pad 2: /3.3V_0.96inch -> /3.3V_OLED
- R8 pad 2: /3.3V_0.96inch -> /3.3V_OLED
- R9 pad 2: /3.3V_0.96inch -> /3.3V_OLED
- U3 pad 2: /3.3V_0.96inch -> /3.3V_OLED
Routing:
- net /3.3V_OLED: track 0.00 -> 47.9 mm, vias 0 -> 2
- net /3.3V_0.96inch: track 47.9 -> 0.00 mm, vias 2 -> 0
Other:
- board text added: "0.96英寸 SPI总线"
- board text added: "分辨率：128×64"
- board text added: "分辨率：160×80"
- board text added: "分辨率：240×240"
- board text added: "分辨率：320×240"
- board text added: "屏幕驱动：ST7735"

Commit message: Update
Parts:
- added ?: LOGO, LOGO, B.Cu at (114.8, 81.2)
- added FPC4: FPC-SMD_10P-0.5mm, Uinio:FPC-SMD_10P-P0.5, F.Cu at (114.9, 75.2)
- FPC1, FPC2: footprint Uinio:FPC-SMD_KH-FG0.5-H2.0-10Pin -> Uinio:FPC-SMD_10P-P0.5
- moved C14 62.8 mm to (120.9, 72.8), turned to 90 degrees
- moved R13 58.3 mm to (120.9, 69.7), turned to -90 degrees
- moved C16 56.5 mm to (114.2, 69.7), turned to 90 degrees
- moved R11 55.9 mm to (118.5, 72.8), turned to 90 degrees
- moved C15 51.1 mm to (109.2, 69.7), turned to 90 degrees
- moved U4 49.8 mm to (111.7, 70.2), turned to 180 degrees
- moved VT3 44.7 mm to (118.5, 70.2)
- moved R12 43.1 mm to (116.1, 69.7), turned to -90 degrees
- moved ? 19.1 mm to (163.8, 130.0)
- moved ? 19.1 mm to (162.5, 89.1)
- moved C1 19.1 mm to (165.6, 100.4)
- moved C10 19.1 mm to (173.5, 124.0)
- moved C11 19.1 mm to (172.3, 124.0)
- moved C13 19.1 mm to (190.6, 124.2)
- moved D1 19.1 mm to (174.6, 121.3)
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Routing:
- net GND: track 119.2 -> 167.8 mm, vias 21 -> 26
- net /3.3V_0.96inch: track 0.00 -> 47.4 mm, vias 0 -> 2
- net /5V_0.96inch: track 0.00 -> 35.9 mm, vias 0 -> 1
- net /SDA_0.96inch: track 0.00 -> 22.5 mm, vias 0 -> 2
- net /SCL_0.96inch: track 0.00 -> 21.0 mm
- net /CS_0.96inch: track 0.00 -> 18.6 mm, vias 0 -> 2
- net /D/C_0.96inch: track 0.00 -> 17.7 mm, vias 0 -> 2
- net /RESET_0.96inch: track 0.00 -> 17.4 mm, vias 0 -> 3
- net /BLK_0.96inch: track 0.00 -> 13.7 mm, vias 0 -> 2
- net Net-(P4-Pad11): track 0.00 -> 13.5 mm, vias 0 -> 2
- net Net-(R11-Pad2): track 0.00 -> 5.27 mm
- net Net-(R13-Pad1): track 0.00 -> 2.45 mm
Other:
- outline, holes or cut-outs redrawn
