File: UINIO-Monitor.kicad_sch (KiCad schematic)
At the start: 38 parts, among them J1 Conn_01x09_Male, J2 Conn_01x09_Male, J3 Conn_01x04_Male, P1 LCD_Pad_10Pin, P2 LCD_Pad_12Pin, P3 OLED_Pad_30Pin, U1 ME6211, U2 ME6211, U3 XC6206PxxxMR

Commit message: Update PCB.
Parts:
- added C? (x3): 1uF, Capacitor_SMD:C_0603_1608Metric, symbol Device:C
- added FPC?: FPC-SMD_10P-0.5mm, Uinio:FPC-SMD_KH-FG0.5-H2.0-10Pin, symbol Uinio:FPC-SMD_10P-0.5mm
- added J?: Conn_01x09_Male, Connector_PinHeader_2.54mm:PinHeader_1x09_P2.54mm_Vertical, symbol Connector:Conn_01x09_Male
- added P?: LCD_Pad_13Pin, Uinio:LCD_Pad_13Pin, symbol Uinio:LCD_Pad_13Pin
- added R?: 10R, Resistor_SMD:R_0603_1608Metric, symbol Device:R
- added R?: 1K, Resistor_SMD:R_0603_1608Metric, symbol Device:R
- added R?: 10K, Resistor_SMD:R_0603_1608Metric, symbol Device:R
- added U?: ME6211, Uinio:SOT-23-5_L3.0-W1.7-P0.95-LS2.8-BR, symbol Uinio:ME6211
- added VT?: S8050, Uinio:SOT-23-3_L2.9-W1.6-P1.90-LS2.9-BL, symbol Uinio:S8050
Connections:
- net 3.3V_0.96inch: now also C?.1, C?.2, FPC?.1, J?.7 (Pin_7), P?.10 (VCC), P?.12 (LEDA), R?.1, U?.5 (Vout)
- net GND: now also C?.1, C?.1, C?.2, FPC?.11, FPC?.12, FPC?.2, FPC?.9, J?.8 (Pin_8), P?.13 (GND2), P?.8 (GND1), U?.2 (Vss), VT?.2 (E)
- net RESET_0.96inch: now also FPC?.6, J?.4 (Pin_4), P?.6 (RESET)
- net SDA_0.96inch: now also FPC?.8, J?.6 (Pin_6), P?.3 (SDA)
- new net: R?.1, R?.2, VT?.1 (B)
- new net: R?.1, VT?.3 (C)
- new net: P?.11 (LEDK), R?.2
- new net 5V_0.96inch: C?.2, FPC?.10, J?.9 (Pin_9), U?.1 (Vin), U?.3 (CE)
- new net BLK_0.96inch: FPC?.3, J?.1 (Pin_1), R?.2
- new net CS_0.96inch: FPC?.4, J?.2 (Pin_2), P?.7 (CS)
- new net D/C_0.96inch: FPC?.5, J?.3 (Pin_3), P?.5 (D/C)
- new net SCL_0.96inch: FPC?.7, J?.5 (Pin_5), P?.4 (SCL)
- no-connect marks 4 -> 8
Other:
- note added: "0.96 英寸 ST7735 LCD 屏幕基板"
- moved on the sheet: C1, C10, C11, C12, C13, C2, C3, C4, C5, C6, C7, C8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

Commit message: Update PCB.
Parts:
- C14, C15, C16: renamed from C?; footprint Capacitor_SMD:C_0603_1608Metric -> Capacitor_SMD:C_0402_1005Metric
- R11, R12, R13: renamed from R?; footprint Resistor_SMD:R_0603_1608Metric -> Resistor_SMD:R_0402_1005Metric
- gave numbers to parts that had none: 5
Connections:
- net 3.3V_0.96inch: no longer C8.2, C9.2, D1.1 (K), FPC3.4, P3.11 (BS1), P3.6 (VBAT), P3.9 (VDD), R7.2, R8.2, R9.2, U3.2 (VO)
- net RESET_0.96inch: no longer C7.2, D1.2 (A), P3.14 (RESET), R7.1
- net SDA_0.96inch: no longer FPC3.2, J3.2 (Pin_2), P3.19 (D1), P3.20 (D2), R9.1
- net SCK_0.96inch renamed SCK_0.96_OLED
- net VCC_0.96inch renamed VCC_0.96_OLED
- new net 3.3V_0.96_OLED: FPC3.4
- new net 3.3V_OLED: C8.2, C9.2, D1.1 (K), P3.11 (BS1), P3.6 (VBAT), P3.9 (VDD), R7.2, R8.2, R9.2, U3.2 (VO)
- new net RESET_0.96_OLED: C7.2, D1.2 (A), P3.14 (RESET), R7.1
- new net SDA_0.96_OLED: FPC3.2, J3.2 (Pin_2), P3.19 (D1), P3.20 (D2), R9.1
Other:
- moved on the sheet: C2, C4, C6, FPC1, J1, P2, R3, R4, R5, U2, VT2

Commit message: Update
Parts:
- removed C9: 0.1uF, Capacitor_SMD:C_0402_1005Metric, symbol Device:C
- removed D1: 1N4148W, Diode_SMD:D_SOD-123, symbol Diode:1N4148W
- added R14: 4.7K, Resistor_SMD:R_0603_1608Metric, symbol Device:R
- C7: value 0.1uF -> 1uF
- FPC1, FPC2, FPC4: footprint Uinio:FPC-SMD_KH-FG0.5-H2.0-10Pin -> Uinio:FPC-SMD_10P-P0.5
- R7, R8, R9: value 10K -> 4.7K; footprint Resistor_SMD:R_0402_1005Metric -> Resistor_SMD:R_0603_1608Metric
Connections:
- net 3.3V_0.96_OLED: now also C8.1, P3.14 (RESET), P3.6 (VBAT), P3.9 (VDD), R7.1, R8.1, U3.2 (VO), R14.1; no longer FPC3.4
- net GND: now also C7.2, C8.2, R9.1; no longer C7.1, C8.1, P3.10 (BS0)
- net SCK_0.96_OLED: now also R7.2; no longer R8.1
- net SDA_0.96_OLED: now also R8.2; no longer R9.1
- removed net 3.3V_OLED: C8.2, P3.11 (BS1), P3.6 (VBAT), P3.9 (VDD), R7.2, R8.2, R9.2, U3.2 (VO)
- removed net RESET_0.96_OLED: C7.2, P3.14 (RESET), R7.1
- net VCC_0.96_OLED: no longer names the net of J3.4 (Pin_4), U3.3 (VI)
- net VCC_0.96_OLED: now also C7.1, FPC3.4
- new net: P3.10 (BS0), R9.2
- new net: P3.11 (BS1), R14.2
Other:
- moved on the sheet: C10, C11, C12, C13, FPC3, J3, P3, R10, U3

Commit message: Finish PCB layout.
Parts:
- R14, R7, R8, R9: footprint Resistor_SMD:R_0603_1608Metric -> Resistor_SMD:R_0402_1005Metric
Other:
- moved on the sheet: C7, C8, FPC3, J3, U3

Commit message: Adding an extension board.
Parts:
- added FPC5: FPC-SMD_4P-0.5mm, Uinio:FPC-SMD_4P-P0.5, symbol Uinio:FPC-SMD_4P-0.5mm
- added FPC6: FPC-SMD_10P-0.5mm, Uinio:FPC-SMD_10P-P0.5, symbol Uinio:FPC-SMD_10P-0.5mm
- added J5: Conn_01x04_Male, Connector_PinHeader_2.54mm:PinHeader_1x04_P2.54mm_Vertical, symbol Connector:Conn_01x04_Male
- added J6: Conn_01x09_Male, Connector_PinHeader_2.54mm:PinHeader_1x09_P2.54mm_Vertical, symbol Connector:Conn_01x09_Male
Connections:
- net GND: now also FPC5.5, FPC5.6, FPC6.11, FPC6.12
- new net: FPC5.1, J5.1 (Pin_1)
- new net: FPC5.2, J5.2 (Pin_2)
- new net: FPC5.3, J5.3 (Pin_3)
- new net: FPC5.4, J5.4 (Pin_4)
- new net: FPC6.3, J6.1 (Pin_1)
- new net: FPC6.4, J6.2 (Pin_2)
- new net: FPC6.5, J6.3 (Pin_3)
- new net: FPC6.6, J6.4 (Pin_4)
- new net: FPC6.7, J6.5 (Pin_5)
- new net: FPC6.8, J6.6 (Pin_6)
- new net: FPC6.1, J6.7 (Pin_7)
- new net: FPC6.2, FPC6.9, J6.8 (Pin_8)
- new net: FPC6.10, J6.9 (Pin_9)
Other:
- note added: "FPC 插座 - 杜邦针转换板"
- moved on the sheet: C10, C11, C12, C13, C2, C4, C6, C7, C8, FPC1, FPC3, J1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

Commit message: Prepare UINIO-Monitor version 2.0.0.
Changed lines of the file:
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@@
     (effects (font (size 1.27 1.27)) (justify left bottom))
+  )
+  (symbol (lib_id "power:GND") (at 306.07 231.14 90) (mirror x) (unit 1)
+    (in_bom yes) (on_board yes)
+    (property "Reference" "#PWR?" (id 0) (at 312.42 231.14 0)
+      (effects (font (size 1.27 1.27)) hide)
+    )
+    (property "Value" "GND" (id 1) (at 309.245 231.14 90)
+      (effects (font (size 1.27 1.27)) (justify right))
+    )
+    (property "Footprint" "" (id 2) (at 306.07 231.14 0)
+      (effects (font (size 1.27 1.27)) hide)
+    )
+    (property "Datasheet" "" (id 3) (at 306.07 231.14 0)
+      (effects (font (size 1.27 1.27)) hide)
+    )
+    (pin "1")
   )
   (symbol (lib_id "power:GND") (at 166.37 34.29 270) (mirror x) (unit 1)
@@
     (pin "2")
   )
+  (symbol (lib_id "power:GND") (at 386.715 238.76 90) (mirror x) (unit 1)
+    (in_bom yes) (on_board yes)
+    (property "Reference" "#PWR?" (id 0) (at 393.065 238.76 0)
+      (effects (font (size 1.27 1.27)) hide)
+    )
+    (property "Value" "GND" (id 1) (at 389.89 238.76 90)
+      (effects (font (size 1.27 1.27)) (justify right))
+    )
+    (property "Footprint" "" (id 2) (at 386.715 238.76 0)
+      (effects (font (size 1.27 1.27)) hide)
+    )
+    (property "Datasheet" "" (id 3) (at 386.715 238.76 0)
+      (effects (font (size 1.27 1.27)) hide)
+    )
+    (pin "1")
+  )
   (symbol (lib_id "Connector:Conn_01x09_Male") (at 30.48 146.685 0) (unit 1)
     (in_bom yes) (on_board yes)
@@
     (pin "1")
   )
-  (symbol (lib_id "power:GND") (at 386.715 238.76 90) (unit 1)
-    (in_bom yes) (on_board yes)
-    (property "Reference" "#PWR040" (id 0) (at 393.065 238.76 0)
-      (effects (font (size 1.27 1.27)) hide)
-    )
-    (property "Value" "GND" (id 1) (at 389.255 238.76 90)
-      (effects (font (size 1.27 1.27)) (justify right))
-    )
-    (property "Footprint" "" (id 2) (at 386.715 238.76 0)
-      (effects (font (size 1.27 1.27)) hide)
-    )
-    (property "Datasheet" "" (id 3) (at 386.715 238.76 0)
-      (effects (font (size 1.27 1.27)) hide)
-    )
-    (pin "1")
-  )
   (symbol (lib_id "Connector:Conn_01x09_Male") (at 344.805 223.52 0) (unit 1)
     (in_bom yes) (on_board yes)
@@
     (pin "1")
   )
-  (symbol (lib_id "power:GND") (at 306.07 208.28 90) (mirror x) (unit 1)
-    (in_bom yes) (on_board yes)
-    (property "Reference" "#PWR037" (id 0) (at 312.42 208.28 0)
-      (effects (font (size 1.27 1.27)) hide)
-    )
-    (property "Value" "GND" (id 1) (at 308.61 208.28 90)
-      (effects (font (size 1.27 1.27)) (justify right))
-    )
-    (property "Footprint" "" (id 2) (at 306.07 208.28 0)
-      (effects (font (size 1.27 1.27)) hide)
-    )
-    (property "Datasheet" "" (id 3) (at 306.07 208.28 0)
-      (effects (font (size 1.27 1.27)) hide)
-    )
-    (pin "1")
-  )
   (symbol (lib_id "power:GND") (at 255.27 224.79 0) (mirror x) (unit 1)
     (in_bom yes) (on_board yes)
@@
     )
     (property "Datasheet" "" (id 3) (at 163.83 214.63 0)
+      (effects (font (size 1.27 1.27)) hide)
+    )
+    (pin "1")
+  )
+  (symbol (lib_id "power:GND") (at 386.715 200.66 90) (mirror x) (unit 1)
+    (in_bom yes) (on_board yes)
+    (property "Reference" "#PWR?" (id 0) (at 393.065 200.66 0)
+      (effects (font (size 1.27 1.27)) hide)
+    )
+    (property "Value" "GND" (id 1) (at 389.89 200.66 90)
+      (effects (font (size 1.27 1.27)) (justify right))
+    )
+    (property "Footprint" "" (id 2) (at 386.715 200.66 0)
+      (effects (font (size 1.27 1.27)) hide)
+    )
+    (property "Datasheet" "" (id 3) (at 386.715 200.66 0)
       (effects (font (size 1.27 1.27)) hide)
     )
@@
     (pin "1")
   )
+  (symbol (lib_id "power:GND") (at 306.07 208.28 90) (mirror x) (unit 1)
+    (in_bom yes) (on_board yes)
+    (property "Reference" "#PWR?" (id 0) (at 312.42 208.28 0)
+      (effects (font (size 1.27 1.27)) hide)
+    )
+    (property "Value" "GND" (id 1) (at 309.245 208.28 90)
+      (effects (font (size 1.27 1.27)) (justify right))
+    )
+    (property "Footprint" "" (id 2) (at 306.07 208.28 0)
+      (effects (font (size 1.27 1.27)) hide)
+    )
+    (property "Datasheet" "" (id 3) (at 306.07 208.28 0)
+      (effects (font (size 1.27 1.27)) hide)
+    )
+    (pin "1")
+  )
   (symbol (lib_id "Device:R") (at 358.775 55.88 90) (unit 1)
     (in_bom yes) (on_board yes)
@@
     (pin "2")
     (pin "3")
-  )
-  (symbol (lib_id "power:GND") (at 386.715 200.66 90) (unit 1)
-    (in_bom yes) (on_board yes)
-    (property "Reference" "#PWR039" (id 0) (at 393.065 200.66 0)
-      (effects (font (size 1.27 1.27)) hide)
-    )
-    (property "Value" "GND" (id 1) (at 389.255 200.66 90)
-      (effects (font (size 1.27 1.27)) (justify right))
-    )
-    (property "Footprint" "" (id 2) (at 386.715 200.66 0)
-      (effects (font (size 1.27 1.27)) hide)
-    )
-    (property "Datasheet" "" (id 3) (at 386.715 200.66 0)
-      (effects (font (size 1.27 1.27)) hide)
-    )
-    (pin "1")
   )
   (symbol (lib_id "power:GND") (at 255.27 137.795 0) (mirror x) (unit 1)
@@
     (pin "5")
   )
-  (symbol (lib_id "power:GND") (at 306.07 231.14 90) (mirror x) (unit 1)
-    (in_bom yes) (on_board yes)
-    (property "Reference" "#PWR038" (id 0) (at 312.42 231.14 0)
-      (effects (font (size 1.27 1.27)) hide)
-    )
-    (property "Value" "GND" (id 1) (at 308.61 231.14 90)
-      (effects (font (size 1.27 1.27)) (justify right))
-    )
-    (property "Footprint" "" (id 2) (at 306.07 231.14 0)
-      (effects (font (size 1.27 1.27)) hide)
-    )
-    (property "Datasheet" "" (id 3) (at 306.07 231.14 0)
-      (effects (font (size 1.27 1.27)) hide)
-    )
-    (pin "1")
-  )
   (symbol (lib_id "Device:R") (at 81.28 135.255 180) (unit 1)
     (in_bom yes) (on_board yes)
@@
       (reference "#PWR036") (unit 1) (value "GND") (footprint "")
     )
-    (path "/68d05bb7-a2dd-4258-ae5c-e9e8ddd5ad14"
-      (reference "#PWR037") (unit 1) (value "GND") (footprint "")
-    )
-    (path "/fb6f3dae-eec4-4e91-8f8a-3b7f2045953a"
-      (reference "#PWR038") (unit 1) (value "GND") (footprint "")
-    )
-    (path "/88b62113-fc96-486a-a238-3c6940674125"
-      (reference "#PWR039") (unit 1) (value "GND") (footprint "")
-    )
-    (path "/43af24d9-ec42-4fac-9950-783879061bdf"
-      (reference "#PWR040") (unit 1) (value "GND") (footprint "")
+    (path "/00440be1-2ecc-46c7-b705-5a3a0a41c2d3"
+      (reference "#PWR?") (unit 1) (value "GND") (footprint "")
+    )
+    (path "/3c33f606-46ce-4c53-b15d-d9cac169ad16"
+      (reference "#PWR?") (unit 1) (value "GND") (footprint "")
+    )
+    (path "/6ec4cc92-d672-4aeb-831c-662af539c466"
+      (reference "#PWR?") (unit 1) (value "GND") (footprint "")
+    )
+    (path "/82e1b127-1b46-4211-872f-c916239465fc"
+      (reference "#PWR?") (unit 1) (value "GND") (footprint "")
     )
     (path "/0efa37a5-698f-4007-a3bb-11fc0938c252"
