File: UINIO-Monitor.kicad_sch (KiCad schematic)
At the start: 52 parts, among them J1 Conn_01x09_Male, J2 Conn_01x09_Male, J3 Conn_01x04_Male, J4 Conn_01x09_Male, J5 Conn_01x04_Male, J6 Conn_01x09_Male, P1 LCD_Pad_10Pin, P2 LCD_Pad_12Pin, P3 OLED_Pad_30Pin, P4 LCD_Pad_13Pin, U1 ME6211, U2 ME6211, U3 XC6206PxxxMR, U4 ME6211

Commit message: Upgrade to Kicad 7.0.0.
Parts:
- removed FPC1, FPC2, FPC4, FPC6: FPC-SMD_10P-0.5mm, Uinio:FPC-SMD_10P-P0.5, symbol Uinio:FPC-SMD_10P-0.5mm
- removed FPC5: FPC-SMD_4P-0.5mm, Uinio:FPC-SMD_4P-P0.5, symbol Uinio:FPC-SMD_4P-0.5mm
- removed J1, J2, J4, J6: Conn_01x09_Male, Connector_PinHeader_2.54mm:PinHeader_1x09_P2.54mm_Vertical, symbol Connector:Conn_01x09_Male
- removed J3, J5: Conn_01x04_Male, Connector_PinHeader_2.54mm:PinHeader_1x04_P2.54mm_Vertical, symbol Connector:Conn_01x04_Male
- added C17, C18, C9: 1uF, Capacitor_SMD:C_0603_1608Metric, symbol Device:C
- added FPC1, FPC2, FPC4, FPC7: FPC-SMD_8P-0.5mm, Uinio:FPC-SMD_8P-P0.5, symbol Uinio:FPC-SMD_8P-0.5mm
- added J1, J2, J4, J7: Conn_01x08_Pin, Connector_PinHeader_2.54mm:PinHeader_1x08_P2.54mm_Vertical, symbol Connector:Conn_01x08_Pin
- added J3: Conn_01x04_Pin, Connector_PinHeader_2.54mm:PinHeader_1x04_P2.54mm_Vertical, symbol Connector:Conn_01x04_Pin
- added P5: LCD_Pad_12Pin, Uinio:LCD_Pad_12Pin, symbol Uinio:LCD_Pad_12Pin
- added R15: 1K, Resistor_SMD:R_0603_1608Metric, symbol Device:R
- added R16: 10K, Resistor_SMD:R_0603_1608Metric, symbol Device:R
- added R17: 10R, Resistor_SMD:R_0603_1608Metric, symbol Device:R
- added U5: ME6211, Uinio:SOT-23-5_L3.0-W1.7-P0.95-LS2.8-BR, symbol Uinio:ME6211
- added VT4: S8050, Uinio:SOT-23-3_L2.9-W1.6-P1.90-LS2.9-BL, symbol Uinio:S8050
Connections:
- net 5V_0.96inch: now also FPC4.8, J4.8 (Pin_8)
- net 5V_2.4inch: now also FPC2.8, J2.8 (Pin_8)
- net BLK_0.96inch: now also FPC4.1, J4.1 (Pin_1)
- net BLK_2.4inch: now also FPC2.1, J2.1 (Pin_1)
- net CS_0.96inch: now also FPC4.2, J4.2 (Pin_2)
- net CS_2.4inch: now also FPC2.2, J2.2 (Pin_2)
- net D/C_0.96inch: now also FPC4.3, J4.3 (Pin_3)
- net D/C_2.4inch: now also FPC2.3, J2.3 (Pin_3)
- net GND: now also C17.1, C18.1, C9.1, FPC1.10, FPC1.7, FPC1.9, FPC2.10, FPC2.7, FPC2.9, FPC4.10, FPC4.7, FPC4.9, FPC7.10, FPC7.7, FPC7.9, J1.7 (Pin_7), J2.7 (Pin_7), J3.3 (Pin_3), J4.7 (Pin_7), J7.7 (Pin_7), P5.1 (GND), P5.12 (GND), P5.5 (GND), P5.6 (GND), U5.2 (Vss), VT4.2 (E)
- net RESET_0.96inch: now also FPC4.4, J4.4 (Pin_4)
- net RESET_2.4inch: now also FPC2.4, J2.4 (Pin_4)
- net SCK_0.96_OLED: now also J3.1 (Pin_1)
- net SCL_0.96inch: now also FPC4.5, J4.5 (Pin_5)
- net SCL_2.4inch: now also FPC2.5, J2.5 (Pin_5)
- net SDA_0.96_OLED: now also J3.2 (Pin_2)
- net SDA_0.96inch: now also FPC4.6, J4.6 (Pin_6)
- net SDA_2.4inch: now also FPC2.6, J2.6 (Pin_6)
- net at C7.1, FPC3.4, U3.3 (VI): now also J3.4 (Pin_4)
- net 3.3V_1.3inch renamed 3.3V_1.33inch
- net 5V_1.3inch renamed 5V_1.33inch
- net 5V_1.33inch: now also FPC1.8, J1.8 (Pin_8)
- net BLK_1.3inch renamed BLK_1.33inch
- net BLK_1.33inch: now also FPC1.1, J1.1 (Pin_1)
- net CS_1.3inch renamed CS_1.33inch
- net CS_1.33inch: now also FPC1.2, J1.2 (Pin_2)
- net D/C_1.3inch renamed D/C_1.33inch
- net D/C_1.33inch: now also FPC1.3, J1.3 (Pin_3)
- net RESET_1.3inch renamed RESET_1.33inch
- net RESET_1.33inch: now also FPC1.4, J1.4 (Pin_4)
- net SCL_1.3inch renamed SCL_1.33inch
- net SCL_1.33inch: now also FPC1.5, J1.5 (Pin_5)
- net SDA_1.3inch renamed SDA_1.33inch
- net SDA_1.33inch: now also FPC1.6, J1.6 (Pin_6)
- new net: R17.1, VT4.3 (C)
- new net: P5.2 (LEDK), R17.2
- new net: R15.1, R16.2, VT4.1 (B)
- new net 3.3V_1.69inch: C18.2, C9.2, P5.3 (LEDA), P5.4 (VDD), R16.1, U5.5 (Vout)
- new net 5V_1.69inch: C17.2, FPC7.8, J7.8 (Pin_8), U5.1 (Vin), U5.3 (CE)
- new net BLK_1.69inch: FPC7.1, J7.1 (Pin_1), R15.2
- new net CS_1.69inch: FPC7.2, J7.2 (Pin_2), P5.8 (CS)
- new net D/C_1.69inch: FPC7.3, J7.3 (Pin_3), P5.7 (D/C)
- new net RESET_1.69inch: FPC7.4, J7.4 (Pin_4), P5.11 (RESET)
- new net SCL_1.69inch: FPC7.5, J7.5 (Pin_5), P5.9 (SCL)
- new net SDA_1.69inch: FPC7.6, J7.6 (Pin_6), P5.10 (SDA)
- no-connect marks 8 -> 9
Other:
- note added: "1.69 英寸 ST7789 LCD 屏幕基板"
- note removed: "FPC 插座 - 杜邦针转换板"
- moved on the sheet: C1, C10, C11, C12, C13, C14, C15, C16, C2, C3, C4, C5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

Commit message: Update PCB.
Parts:
- added C19: 10uF, Capacitor_SMD:C_0402_1005Metric, symbol Device:C
- added D2: SS14, Uinio:SMA_L4.3-W2.5-LS5.0-RD, symbol Uinio:SS14
- added R18, R19, R20: 4.7K, Resistor_SMD:R_0402_1005Metric, symbol Device:R
Connections:
- net 3.3V_0.96_OLED: now also D2.1 (K), R18.2, R19.2; no longer P3.14 (RESET)
- net GND: now also C19.2, R20.2; no longer P3.15 (D/C)
- new net D/C: P3.15 (D/C), R19.1, R20.1
- new net RESET: C19.1, D2.2 (A), P3.14 (RESET), R18.1
Other:
- note added: "I²C 地址选择"
- note added: "上拉地址：0x7A"
- note added: "下拉地址：0x78"
- note added: "复位逻辑"
- moved on the sheet: C10, C11, C12, C13, C7, C8, FPC3, J3, P3, R10, R14, R7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

Commit message: Update PCB.
Parts:
- removed D2: SS14, Uinio:SMA_L4.3-W2.5-LS5.0-RD, symbol Uinio:SS14
- removed R14, R9: 4.7K, Resistor_SMD:R_0402_1005Metric, symbol Device:R
- added D1: 1N5819, Diode_SMD:D_SOD-323F, symbol Diode:1N5819
- C7: value 1uF -> 0.1uF
Connections:
- net 3.3V_0.96_OLED: now also P3.11 (BS1), D1.1 (K)
- net GND: now also P3.10 (BS0)
- net RESET: now also D1.2 (A)
